Commit message: omni running

File: mishanya_description/urdf/base.xacro (robot description, xacro)
@@ -3,9 +3,6 @@
   <xacro:property name="M_PI" value="3.1415926535897931" />
   <!-- base property -->
-  <xacro:property name="base_mass" value="1" />
-  <xacro:property name="base_length" value="0.81" />
-  <xacro:property name="base_width" value="0.81" />
   <xacro:property name="base_height" value="0.21" />
-  <xacro:property name="base_mass" value="10" />
+  <xacro:property name="base_mass" value="2" />
   <xacro:property name="base_rad" value="0.4" />
   <xacro:property name="base_length" value="0.21" />
@@ -23,7 +20,8 @@
   </xacro:macro>
   <!-- inertial macros -->
+  <link name="origin_link"/>
   <link name="base_link">
     <collision name="collision_chassis">
-      <origin rpy="0 0 0" xyz="0 0 0.1"/>
+      <origin rpy="0 0 0" xyz="0 0 0.15"/>
       <geometry>
         <cylinder length="${base_length}" radius="${base_rad}"/>
@@ -31,5 +29,5 @@
     </collision>
     <visual>
-      <origin rpy="0 0 0" xyz="0 0 0.1"/>
+      <origin rpy="0 0 0" xyz="0 0 0.15"/>
       <geometry>
         <cylinder length="${base_length}" radius="${base_rad}"/>

File: mishanya_description/urdf/kernel.xacro (robot description, xacro)
@@ -3,6 +3,6 @@
   <!-- kernel property -->
   <xacro:property name="kernel_mass" value="1" />
-  <xacro:property name="kernel_rad" value="0.05" />
-  <xacro:property name="kernel_length" value="1" />
+  <xacro:property name="kernel_rad" value="0.03" />
+  <xacro:property name="kernel_length" value="0.053" />
   <!-- kernel property -->
   <!-- inertial macros -->
@@ -26,5 +26,5 @@
       </xacro:solid_cylinder_inertial>
       <collision name="link_kernel_collision">
-        <origin rpy="0 0 0" xyz="0 0 0"/>
+        <origin rpy="0 0 0" xyz="0 0 ${kernel_length/2}"/>
         <geometry>
           <cylinder length="${kernel_length}" radius="${kernel_rad}"/>
@@ -32,5 +32,5 @@
       </collision>
       <visual name="${name}_visual">
-        <origin rpy="0 0 0" xyz="0 0 0"/>
+        <origin rpy="0 0 0" xyz="0 0 ${kernel_length/2}"/>
         <geometry>
           <cylinder length="${kernel_length}" radius="${kernel_rad}"/>

File: mishanya_description/urdf/mishanya.xacro (robot description, xacro)
@@ -1,8 +1,41 @@
 <?xml version="1.0" ?>
 <robot name="mishanya" xmlns:xacro="http://www.ros.org/wiki/xacro">
-  <xacro:include filename="$(find mishanya_description)/urdf/omni.xacro" />
+  <xacro:include filename="$(find mishanya_description)/urdf/rim.xacro"/>
   <xacro:include filename="$(find mishanya_description)/urdf/kernel.xacro" />
   <xacro:include filename="$(find mishanya_description)/urdf/base.xacro" />
-  <xacro:link_kernel name="kernel" />
-	<xacro:joint_kernel name="joint_kernel" child="kernel" origin_xyz="0 0 ${2*base_height}" />
+	<joint
+		name="base_joint"
+		type="fixed"
+	>
+		<parent link="origin_link" />
+		<child link="base_link" />
+		<origin
+			xyz="0 0 0.01905"
+		/>
+	</joint>
+	<xacro:rim_macro
+		name="left"
+		color="0.3 0 0"
+		xyz="-0.3464101615 0.2 0"
+		rpy="1.570796326794896 0 1.047197551196597"
+	/>
+	<xacro:rim_macro
+		name="back"
+		color="0 0.3 0"
+		xyz="0 -0.4 0"
+		rpy="1.570796326794896 0 3.141592653589793"
+	/>
+	<xacro:rim_macro
+		name="right"
+		color="0 0 0.3"
+		xyz="0.3464101615 0.2 0"
+		rpy="1.570796326794896 0 -1.047197551196597"
+	/>
+  <!-- <xacro:link_kernel name="kernel" />
+	<xacro:joint_kernel name="joint_kernel" child="kernel" origin_xyz="0 0 ${base_height}" /> -->
+  <gazebo>
+		<plugin name="gazebo_ros_control" filename="libgazebo_ros_control.so">
+			<robotNamespace>/open_base</robotNamespace>
+		</plugin>
+	</gazebo>
  </robot>

Commit message: add twist key

File: mishanya_description/urdf/base.xacro (robot description, xacro)
@@ -4,5 +4,5 @@
   <!-- base property -->
   <xacro:property name="base_height" value="0.21" />
-  <xacro:property name="base_mass" value="2" />
+  <xacro:property name="base_mass" value="5" />
   <xacro:property name="base_rad" value="0.4" />
   <xacro:property name="base_length" value="0.21" />
@@ -23,5 +23,5 @@
   <link name="base_link">
     <collision name="collision_chassis">
-      <origin rpy="0 0 0" xyz="0 0 0.15"/>
+      <origin rpy="0 0 0" xyz="0 0 0.1"/>
       <geometry>
         <cylinder length="${base_length}" radius="${base_rad}"/>
@@ -29,5 +29,5 @@
     </collision>
     <visual>
-      <origin rpy="0 0 0" xyz="0 0 0.15"/>
+      <origin rpy="0 0 0" xyz="0 0 0.1"/>
       <geometry>
         <cylinder length="${base_length}" radius="${base_rad}"/>

File: mishanya_description/urdf/kernel.xacro (robot description, xacro)
@@ -2,7 +2,7 @@
 <robot xmlns:xacro="http://www.ros.org/wiki/xacro">
   <!-- kernel property -->
-  <xacro:property name="kernel_mass" value="1" />
+  <xacro:property name="kernel_mass" value="0.5" />
   <xacro:property name="kernel_rad" value="0.03" />
-  <xacro:property name="kernel_length" value="0.053" />
+  <xacro:property name="kernel_length" value="0.53" />
   <!-- kernel property -->
   <!-- inertial macros -->

File: mishanya_description/urdf/mishanya.xacro (robot description, xacro)
@@ -32,6 +32,6 @@
 		rpy="1.570796326794896 0 -1.047197551196597"
 	/>
-  <!-- <xacro:link_kernel name="kernel" />
-	<xacro:joint_kernel name="joint_kernel" child="kernel" origin_xyz="0 0 ${base_height}" /> -->
+  <xacro:link_kernel name="kernel" />
+	<xacro:joint_kernel name="joint_kernel" child="kernel" origin_xyz="0 0 ${base_height}" />
   <gazebo>
 		<plugin name="gazebo_ros_control" filename="libgazebo_ros_control.so">

File: mishanya_description/urdf/rim.xacro (robot description, xacro)
@@ -9,5 +9,5 @@
 			<inertial>
 				<origin xyz="0 0 -0.000343"/>
-				<mass value="0.835758"/>
+				<mass value="1.835758"/>
 				<inertia
 					ixx="6.63684e-07"

Commit message: first sim with webots

File: mishanya_description/urdf/base.xacro (robot description, xacro)
@@ -1,5 +1,4 @@
 <?xml version="1.0"?>
 <robot xmlns:xacro="http://www.ros.org/wiki/xacro">
-  <xacro:property name="M_PI" value="3.1415926535897931" />
   <!-- base property -->
   <xacro:property name="base_height" value="0.21" />
@@ -20,23 +19,22 @@
   </xacro:macro>
   <!-- inertial macros -->
-  <link name="origin_link"/>
-  <link name="base_link">
-    <collision name="collision_chassis">
-      <origin rpy="0 0 0" xyz="0 0 0.1"/>
-      <geometry>
-        <cylinder length="${base_length}" radius="${base_rad}"/>
-      </geometry>
-    </collision>
-    <visual>
-      <origin rpy="0 0 0" xyz="0 0 0.1"/>
-      <geometry>
-        <cylinder length="${base_length}" radius="${base_rad}"/>
-      </geometry>
-    </visual>
-    <xacro:solid_cylinder_inertial
-          r="${base_rad}" h="${base_length}"
-          mass="${base_mass}">
-      <origin xyz="0 0 0" rpy="0 0 0" />
-    </xacro:solid_cylinder_inertial>
-  </link>
+    <link name="base_link">
+      <collision name="collision_chassis">
+        <origin rpy="0 0 0" xyz="0 0 0.1"/>
+        <geometry>
+          <cylinder length="${base_length}" radius="${base_rad}"/>
+        </geometry>
+      </collision>
+      <visual>
+        <origin rpy="0 0 0" xyz="0 0 0.1"/>
+        <geometry>
+          <cylinder length="${base_length}" radius="${base_rad}"/>
+        </geometry>
+      </visual>
+      <xacro:solid_cylinder_inertial
+            r="${base_rad}" h="${base_length}"
+            mass="${base_mass}">
+        <origin xyz="0 0 0" rpy="0 0 0" />
+      </xacro:solid_cylinder_inertial>
+    </link>
 </robot>

File: mishanya_description/urdf/mishanya.xacro (robot description, xacro)
@@ -1,41 +1,7 @@
-<?xml version="1.0" ?>
+<?xml version="1.0"?>
 <robot name="mishanya" xmlns:xacro="http://www.ros.org/wiki/xacro">
-  <xacro:include filename="$(find mishanya_description)/urdf/rim.xacro"/>
   <xacro:include filename="$(find mishanya_description)/urdf/kernel.xacro" />
   <xacro:include filename="$(find mishanya_description)/urdf/base.xacro" />
-	<joint
-		name="base_joint"
-		type="fixed"
-	>
-		<parent link="origin_link" />
-		<child link="base_link" />
-		<origin
-			xyz="0 0 0.01905"
-		/>
-	</joint>
-	<xacro:rim_macro
-		name="left"
-		color="0.3 0 0"
-		xyz="-0.3464101615 0.2 0"
-		rpy="1.570796326794896 0 1.047197551196597"
-	/>
-	<xacro:rim_macro
-		name="back"
-		color="0 0.3 0"
-		xyz="0 -0.4 0"
-		rpy="1.570796326794896 0 3.141592653589793"
-	/>
-	<xacro:rim_macro
-		name="right"
-		color="0 0 0.3"
-		xyz="0.3464101615 0.2 0"
-		rpy="1.570796326794896 0 -1.047197551196597"
-	/>
   <xacro:link_kernel name="kernel" />
-	<xacro:joint_kernel name="joint_kernel" child="kernel" origin_xyz="0 0 ${base_height}" />
-  <gazebo>
-		<plugin name="gazebo_ros_control" filename="libgazebo_ros_control.so">
-			<robotNamespace>/open_base</robotNamespace>
-		</plugin>
-	</gazebo>
- </robot>
+	<xacro:joint_kernel name="joint_kernel" child="kernel" origin_xyz="0 0 ${2*base_height}" />
+</robot>

Commit message: webots sim with omni wheels

File: mishanya_description/urdf/base.xacro (robot description, xacro)
@@ -21,5 +21,5 @@
     <link name="base_link">
       <collision name="collision_chassis">
-        <origin rpy="0 0 0" xyz="0 0 0.1"/>
+        <origin rpy="0 0 0" xyz="0 0 0"/>
         <geometry>
           <cylinder length="${base_length}" radius="${base_rad}"/>
@@ -27,5 +27,5 @@
       </collision>
       <visual>
-        <origin rpy="0 0 0" xyz="0 0 0.1"/>
+        <origin rpy="0 0 0" xyz="0 0 0"/>
         <geometry>
           <cylinder length="${base_length}" radius="${base_rad}"/>

File: mishanya_description/urdf/mishanya.urdf (robot description, URDF)
Before this commit: robot mishanya, 2 links, 1 joints
Links:
- added link back_left_wheel_link; collision cylinder length=0.00435 radius=0.0635; visual mesh filename=package://summit_description/meshes/wheels/omni_wheel_2.dae scale=0.5 0.5 0.5
- added link back_right_wheel_link; collision cylinder length=0.00435 radius=0.0635; visual mesh filename=package://summit_description/meshes/wheels/omni_wheel_2.dae scale=0.5 0.5 0.5
- added link base_footprint; visual box size=0.001 0.001 0.001
- added link front_wheel_link; collision cylinder length=0.00435 radius=0.0635; visual mesh filename=package://summit_description/meshes/wheels/omni_wheel_2.dae scale=0.5 0.5 0.5
Joints:
- added joint back_left_wheel_joint: type continuous, parent base_link, child back_left_wheel_link, origin xyz=-0.282842712474619 0.282842712474619 -0.105 rpy=0 0 0.7853981633974483, axis 0 1 0, limit effort=100 velocity=100
- added joint back_right_wheel_joint: type continuous, parent base_link, child back_right_wheel_link, origin xyz=-0.282842712474619 -0.282842712474619  -0.105 rpy=0 0 -0.7853981633974483, axis 0 1 0, limit effort=100 velocity=100
- added joint base_footprint_joint: type fixed, parent base_footprint, child base_link, origin xyz=0 0 0.16849999999999998 rpy=0 0 0
- added joint front_wheel_joint: type continuous, parent base_link, child front_wheel_link, origin xyz=0.4 0 -0.105 rpy=0 0 1.5707963267948966, axis 0 1 0, limit effort=100 velocity=100
- joint joint_kernel: axis 0 0 0.42 -> 0 0 0.105; origin xyz=0 0 0.42 rpy=0 0 0 -> xyz=0 0 0.105 rpy=0 0 0

File: mishanya_description/urdf/mishanya.xacro (robot description, xacro)
@@ -3,5 +3,29 @@
   <xacro:include filename="$(find mishanya_description)/urdf/kernel.xacro" />
   <xacro:include filename="$(find mishanya_description)/urdf/base.xacro" />
+  <xacro:include filename="$(find mishanya_description)/urdf/omni_wheel.xacro" />
+  <xacro:property name="M_PI" value="3.1415926535897931" />
+  <link name="base_footprint">
+    <visual>
+      <origin xyz="0 0 0" rpy="0 0 0" />
+      <geometry>
+        <box size="0.001 0.001 0.001" />
+      </geometry>
+    </visual>
+  </link>
+  <joint name="base_footprint_joint" type="fixed">
+    <origin xyz="0 0 ${wheel_radius + base_height/2}" rpy="0 0 0" />
+    <parent link="base_footprint"/>
+    <child link="base_link" />
+  </joint>
   <xacro:link_kernel name="kernel" />
-	<xacro:joint_kernel name="joint_kernel" child="kernel" origin_xyz="0 0 ${2*base_height}" />
+	<xacro:joint_kernel name="joint_kernel" child="kernel" origin_xyz="0 0 ${base_height/2}" />
+  <xacro:omni_wheel prefix="front" parent="base_link" reflect="false">
+    <origin xyz="${base_rad} 0 -${base_height/2}" rpy="0 0 ${M_PI/2}"/>
+  </xacro:omni_wheel>
+  <xacro:omni_wheel prefix="back_left" parent="base_link" reflect="false">
+    <origin xyz="-${base_rad/sqrt(2)} ${base_rad/sqrt(2)} -${base_height/2}" rpy="0 0 ${M_PI/4}"/>
+  </xacro:omni_wheel>
+  <xacro:omni_wheel prefix="back_right" parent="base_link" reflect="false">
+    <origin xyz="-${base_rad/sqrt(2)} -${base_rad/sqrt(2)}  -${base_height/2}" rpy="0 0 -${M_PI/4}"/>
+  </xacro:omni_wheel>
 </robot>
